Commit message: Enhance Haller robot with vision capabilities; update navigation parameters to include vision layers for obstacle detection and traversability, modify camera properties in URDF, and improve launch files for hardware and simulation to support vision processing.

File: src/haller_ros/haller_common/haller_description/urdf/gazebo_plugins.xacro (robot description, xacro)
@@ -45,5 +45,6 @@
       </sensor>
     </gazebo>
-    <!-- Camera plugin -->
+    <!-- Camera plugin (IMX219 J8IM228-V3.0 simulation) -->
+    <!-- Matches hardware: 120° FOV, 640x480 @ 30fps for inference -->
     <gazebo reference="camera_link">
       <sensor name="camera" type="camera">
@@ -52,6 +53,8 @@
         <update_rate>30</update_rate>
         <camera name="front_camera">
-          <horizontal_fov>1.3962634</horizontal_fov>
+          <!-- 120 degrees FOV = 2.0944 radians -->
+          <horizontal_fov>2.0944</horizontal_fov>
           <image>
+            <!-- Resolution optimized for inference on Orin Nano 8GB -->
             <width>640</width>
             <height>480</height>
@@ -62,4 +65,13 @@
             <far>100</far>
           </clip>
+          <distortion>
+            <!-- IMX219 with wide-angle lens has some barrel distortion -->
+            <k1>-0.25</k1>
+            <k2>0.12</k2>
+            <k3>0.0</k3>
+            <p1>0.0</p1>
+            <p2>0.0</p2>
+            <center>0.5 0.5</center>
+          </distortion>
           <noise>
             <type>gaussian</type>
@@ -70,4 +82,5 @@
         <plugin name="camera_controller" filename="libgazebo_ros_camera.so">
           <ros>
+            <!-- Unified topic names for sim/hardware abstraction -->
             <remapping>~/image_raw:=camera/image_raw</remapping>
             <remapping>~/camera_info:=camera/camera_info</remapping>
@@ -75,5 +88,5 @@
           <camera_name>camera</camera_name>
           <frame_name>camera_optical_frame</frame_name>
-          <hack_baseline>0.07</hack_baseline>
+          <hack_baseline>0.0</hack_baseline>
         </plugin>
       </sensor>

File: src/haller_ros/haller_common/haller_description/urdf/haller_sensors.xacro (robot description, xacro)
@@ -9,7 +9,11 @@
   <xacro:property name="lidar_height" value="0.04"/>
   <xacro:property name="lidar_mass" value="0.2"/>
-  <!-- Camera properties -->
-  <xacro:property name="camera_size" value="0.03"/>
-  <xacro:property name="camera_mass" value="0.1"/>
+  <!-- Camera properties (IMX219 J8IM228-V3.0 module) -->
+  <!-- Module dimensions: ~25mm x 24mm x 9mm -->
+  <xacro:property name="camera_width" value="0.025"/>   <!-- X: depth/forward -->
+  <xacro:property name="camera_height" value="0.024"/>  <!-- Y: width -->
+  <xacro:property name="camera_depth" value="0.009"/>   <!-- Z: height -->
+  <xacro:property name="camera_mass" value="0.003"/>    <!-- ~3 grams -->
+  <!-- FOV: 120 degrees = 2.0944 radians (configured in gazebo_plugins.xacro) -->
   <xacro:macro name="haller_sensors">
     <!-- ==================== LiDAR Sensor ==================== -->
@@ -48,10 +52,11 @@
       <material>Gazebo/Black</material>
     </gazebo>
-    <!-- ==================== Front Camera ==================== -->
+    <!-- ==================== Front Camera (IMX219 J8IM228-V3.0) ==================== -->
+    <!-- 120° FOV CSI camera module for Jetson Orin -->
     <link name="camera_link">
       <visual>
         <origin xyz="0 0 0" rpy="0 0 0"/>
         <geometry>
-          <box size="${camera_size} ${camera_size * 2} ${camera_size}"/>
+          <box size="${camera_width} ${camera_height} ${camera_depth}"/>
         </geometry>
         <material name="dark_grey"/>
@@ -60,9 +65,9 @@
         <origin xyz="0 0 0" rpy="0 0 0"/>
         <geometry>
-          <box size="${camera_size} ${camera_size * 2} ${camera_size}"/>
+          <box size="${camera_width} ${camera_height} ${camera_depth}"/>
         </geometry>
       </collision>
       <xacro:box_inertial mass="${camera_mass}"
-        x="${camera_size}" y="${camera_size * 2}" z="${camera_size}">
+        x="${camera_width}" y="${camera_height}" z="${camera_depth}">
         <origin xyz="0 0 0" rpy="0 0 0"/>
       </xacro:box_inertial>
