Commit message: Pre-JetPack-7 snapshot: motor/URDF/controller/install tuning

File: src/haller_ros/haller_common/haller_description/urdf/haller_base.xacro (robot description, xacro)
@@ -1,7 +1,8 @@
 <?xml version="1.0"?>
 <robot xmlns:xacro="http://www.ros.org/wiki/xacro">
-  <!-- Robot Dimensions -->
-  <xacro:property name="chassis_length" value="0.40"/>
-  <xacro:property name="chassis_width" value="0.30"/>
+  <!-- Robot Dimensions (triangular chassis approximated as a box) -->
+  <!-- Two driven wheels in front (35cm apart), castor 27cm behind -->
+  <xacro:property name="chassis_length" value="0.27"/>
+  <xacro:property name="chassis_width" value="0.35"/>
   <xacro:property name="chassis_height" value="0.15"/>
   <xacro:property name="chassis_mass" value="10.0"/>
@@ -14,5 +15,5 @@
     <link name="chassis_link">
       <visual>
-        <origin xyz="0 0 ${chassis_z_offset}" rpy="0 0 0"/>
+        <origin xyz="${-chassis_length/2} 0 ${chassis_z_offset}" rpy="0 0 0"/>
         <geometry>
           <box size="${chassis_length} ${chassis_width} ${chassis_height}"/>
@@ -21,5 +22,5 @@
       </visual>
       <collision>
-        <origin xyz="0 0 ${chassis_z_offset}" rpy="0 0 0"/>
+        <origin xyz="${-chassis_length/2} 0 ${chassis_z_offset}" rpy="0 0 0"/>
         <geometry>
           <box size="${chassis_length} ${chassis_width} ${chassis_height}"/>
@@ -28,5 +29,5 @@
       <xacro:box_inertial mass="${chassis_mass}"
         x="${chassis_length}" y="${chassis_width}" z="${chassis_height}">
-        <origin xyz="0 0 ${chassis_z_offset}" rpy="0 0 0"/>
+        <origin xyz="${-chassis_length/2} 0 ${chassis_z_offset}" rpy="0 0 0"/>
       </xacro:box_inertial>
     </link>
@@ -59,5 +60,5 @@
       <parent link="chassis_link"/>
       <child link="top_plate_link"/>
-      <origin xyz="0 0 ${chassis_z_offset + chassis_height/2 + top_plate_height/2}" rpy="0 0 0"/>
+      <origin xyz="${-chassis_length/2} 0 ${chassis_z_offset + chassis_height/2 + top_plate_height/2}" rpy="0 0 0"/>
     </joint>
   </xacro:macro>

File: src/haller_ros/haller_common/haller_description/urdf/haller_ros2_control.xacro (robot description, xacro)
@@ -29,6 +29,6 @@
         </xacro:unless>
       </xacro:unless>
-      <!-- Front Left Wheel -->
-      <joint name="front_left_wheel_joint">
+      <!-- Left Wheel -->
+      <joint name="left_wheel_joint">
         <command_interface name="velocity">
           <param name="min">-10</param>
@@ -38,24 +38,6 @@
         <state_interface name="velocity"/>
       </joint>
-      <!-- Front Right Wheel -->
-      <joint name="front_right_wheel_joint">
-        <command_interface name="velocity">
-          <param name="min">-10</param>
-          <param name="max">10</param>
-        </command_interface>
-        <state_interface name="position"/>
-        <state_interface name="velocity"/>
-      </joint>
-      <!-- Rear Left Wheel -->
-      <joint name="rear_left_wheel_joint">
-        <command_interface name="velocity">
-          <param name="min">-10</param>
-          <param name="max">10</param>
-        </command_interface>
-        <state_interface name="position"/>
-        <state_interface name="velocity"/>
-      </joint>
-      <!-- Rear Right Wheel -->
-      <joint name="rear_right_wheel_joint">
+      <!-- Right Wheel -->
+      <joint name="right_wheel_joint">
         <command_interface name="velocity">
           <param name="min">-10</param>

File: src/haller_ros/haller_common/haller_description/urdf/haller_wheels.xacro (robot description, xacro)
@@ -5,10 +5,12 @@
   <xacro:property name="wheel_width" value="0.04"/>
   <xacro:property name="wheel_mass" value="0.5"/>
-  <!-- Wheel positions -->
-  <xacro:property name="wheel_x_offset" value="0.13"/>
-  <xacro:property name="wheel_y_offset" value="0.17"/>
-  <xacro:property name="wheel_z_offset" value="0.0"/>
-  <!-- Wheel macro -->
-  <xacro:macro name="wheel" params="prefix x_reflect y_reflect">
+  <!-- Wheel positions (drive wheels at base_link origin line) -->
+  <xacro:property name="wheel_y_offset" value="0.175"/>  <!-- half of 0.35m separation -->
+  <!-- Castor wheel properties -->
+  <xacro:property name="castor_radius" value="0.025"/>
+  <xacro:property name="castor_mass" value="0.1"/>
+  <xacro:property name="castor_x_offset" value="-0.27"/>  <!-- behind drive axle -->
+  <!-- Drive wheel macro -->
+  <xacro:macro name="drive_wheel" params="prefix y_reflect">
     <link name="${prefix}_wheel_link">
       <visual>
@@ -33,11 +35,8 @@
       <parent link="base_link"/>
       <child link="${prefix}_wheel_link"/>
-      <origin
-        xyz="${x_reflect * wheel_x_offset} ${y_reflect * wheel_y_offset} ${wheel_z_offset}"
-        rpy="0 0 0"/>
+      <origin xyz="0 ${y_reflect * wheel_y_offset} 0" rpy="0 0 0"/>
       <axis xyz="0 1 0"/>
       <dynamics damping="0.1" friction="0.1"/>
     </joint>
-    <!-- Gazebo wheel properties -->
     <gazebo reference="${prefix}_wheel_link">
       <material>Gazebo/DarkGrey</material>
@@ -52,10 +51,40 @@
   <!-- All wheels macro -->
   <xacro:macro name="haller_wheels">
-    <!-- Front wheels -->
-    <xacro:wheel prefix="front_left" x_reflect="1" y_reflect="1"/>
-    <xacro:wheel prefix="front_right" x_reflect="1" y_reflect="-1"/>
-    <!-- Rear wheels -->
-    <xacro:wheel prefix="rear_left" x_reflect="-1" y_reflect="1"/>
-    <xacro:wheel prefix="rear_right" x_reflect="-1" y_reflect="-1"/>
+    <!-- Drive wheels (at the front, on the drive axle) -->
+    <xacro:drive_wheel prefix="left" y_reflect="1"/>
+    <xacro:drive_wheel prefix="right" y_reflect="-1"/>
+    <!-- Castor wheel (rear) -->
+    <link name="castor_wheel_link">
+      <visual>
+        <origin xyz="0 0 0" rpy="0 0 0"/>
+        <geometry>
+          <sphere radius="${castor_radius}"/>
+        </geometry>
+        <material name="dark_grey"/>
+      </visual>
+      <collision>
+        <origin xyz="0 0 0" rpy="0 0 0"/>
+        <geometry>
+          <sphere radius="${castor_radius}"/>
+        </geometry>
+      </collision>
+      <xacro:sphere_inertial mass="${castor_mass}" radius="${castor_radius}">
+        <origin xyz="0 0 0" rpy="0 0 0"/>
+      </xacro:sphere_inertial>
+    </link>
+    <joint name="castor_wheel_joint" type="fixed">
+      <parent link="base_link"/>
+      <child link="castor_wheel_link"/>
+      <origin xyz="${castor_x_offset} 0 ${-(wheel_radius - castor_radius)}" rpy="0 0 0"/>
+    </joint>
+    <gazebo reference="castor_wheel_link">
+      <material>Gazebo/Grey</material>
+      <mu1>0.0</mu1>
+      <mu2>0.0</mu2>
+      <kp>1000000.0</kp>
+      <kd>100.0</kd>
+      <minDepth>0.001</minDepth>
+      <maxVel>1.0</maxVel>
+    </gazebo>
   </xacro:macro>
 </robot>
