Commit message: fix(base): 3-wheel diff-drive (2 front + rear caster), not 4-wheel
Correct the base across docs, HMI, and the robot description. README/src/docs/BasePanel said '4-wheel'; the URDF modelled 4 wheels as skid-steer. Now: 2 driven front wheels + a passive frictionless rear caster; ros2_control drops the rear joints; controller left/right_wheel_names = one wheel each. XML/YAML valid; not yet colcon-built/xacro-expanded/sim-tested.

File: src/haller_ros/haller_common/haller_description/urdf/haller_ros2_control.xacro (robot description, xacro)
@@ -47,22 +47,6 @@
         <state_interface name="velocity"/>
       </joint>
-      <!-- Rear Left Wheel -->
-      <joint name="rear_left_wheel_joint">
-        <command_interface name="velocity">
-          <param name="min">-10</param>
-          <param name="max">10</param>
-        </command_interface>
-        <state_interface name="position"/>
-        <state_interface name="velocity"/>
-      </joint>
-      <!-- Rear Right Wheel -->
-      <joint name="rear_right_wheel_joint">
-        <command_interface name="velocity">
-          <param name="min">-10</param>
-          <param name="max">10</param>
-        </command_interface>
-        <state_interface name="position"/>
-        <state_interface name="velocity"/>
-      </joint>
+      <!-- No rear wheel joints: the rear is a passive caster (see haller_wheels.xacro),
+           not an actuated wheel. Differential drive = 2 driven front wheels. -->
     </ros2_control>
   </xacro:macro>

File: src/haller_ros/haller_common/haller_description/urdf/haller_wheels.xacro (robot description, xacro)
@@ -50,12 +50,55 @@
     </gazebo>
   </xacro:macro>
-  <!-- All wheels macro -->
+  <!-- Passive rear caster: the 3rd contact point of the differential-drive
+       base (2 driven front wheels + this caster). Modelled as a frictionless
+       sphere fixed to base_link so it slides freely while the front wheels steer. -->
+  <xacro:property name="caster_radius" value="${wheel_radius}"/>
+  <xacro:property name="caster_x_offset" value="0.13"/>
+  <xacro:property name="caster_mass" value="0.2"/>
+  <xacro:macro name="rear_caster">
+    <link name="rear_caster_link">
+      <visual>
+        <origin xyz="0 0 0" rpy="0 0 0"/>
+        <geometry>
+          <sphere radius="${caster_radius}"/>
+        </geometry>
+        <material name="black"/>
+      </visual>
+      <collision>
+        <origin xyz="0 0 0" rpy="0 0 0"/>
+        <geometry>
+          <sphere radius="${caster_radius}"/>
+        </geometry>
+      </collision>
+      <inertial>
+        <mass value="${caster_mass}"/>
+        <origin xyz="0 0 0" rpy="0 0 0"/>
+        <!-- solid sphere: I = 2/5 m r^2 -->
+        <inertia ixx="${0.4 * caster_mass * caster_radius * caster_radius}" ixy="0.0" ixz="0.0"
+                 iyy="${0.4 * caster_mass * caster_radius * caster_radius}" iyz="0.0"
+                 izz="${0.4 * caster_mass * caster_radius * caster_radius}"/>
+      </inertial>
+    </link>
+    <joint name="rear_caster_joint" type="fixed">
+      <parent link="base_link"/>
+      <child link="rear_caster_link"/>
+      <origin xyz="${-caster_x_offset} 0 ${wheel_z_offset}" rpy="0 0 0"/>
+    </joint>
+    <!-- Frictionless in Gazebo so the caster doesn't fight the diff-drive. -->
+    <gazebo reference="rear_caster_link">
+      <material>Gazebo/DarkGrey</material>
+      <mu1>0.0</mu1>
+      <mu2>0.0</mu2>
+      <kp>1000000.0</kp>
+      <kd>100.0</kd>
+      <minDepth>0.001</minDepth>
+      <maxVel>1.0</maxVel>
+    </gazebo>
+  </xacro:macro>
+  <!-- All wheels macro: 2 driven front wheels + 1 passive rear caster -->
   <xacro:macro name="haller_wheels">
-    <!-- Front wheels -->
     <xacro:wheel prefix="front_left" x_reflect="1" y_reflect="1"/>
     <xacro:wheel prefix="front_right" x_reflect="1" y_reflect="-1"/>
-    <!-- Rear wheels -->
-    <xacro:wheel prefix="rear_left" x_reflect="-1" y_reflect="1"/>
-    <xacro:wheel prefix="rear_right" x_reflect="-1" y_reflect="-1"/>
+    <xacro:rear_caster/>
   </xacro:macro>
 </robot>
